File: Hardware/Electrical/Adafruit Servo HAT rev A.sch (EAGLE design)
At the start: 51 parts, among them Q1 AOD417, U1 CAT24C32, U2 PCA9685, X1 2.1mm SMT

Commit message: PCB Designs
Parts:
- removed 5-PIN-HEAD: (no value), pinhead:PINHD-1X5
- removed D1_OPEN, D1_STATE, D2_OPEN, D2_STATE, LVR_FOOD: (no value), adafruit:JST_2PIN-SMT
- removed DISPENSER, DOOR1, DOOR2, LVR_DISPENSER: SERVO, SparkFun-Electromechanical:SERVO
- removed IR1, IR2, READ_PELLET: (no value), adafruit:JST_3PIN
- added FID1, FID2, FID3: FIDUCIAL"", microbuilder:FIDUCIAL""
Connections:
- removed net N$1: R1.2, R2.2, U1.VCC
- net +5V: no longer DISPENSER.V+, DOOR1.V+, DOOR2.V+, IR1.2, IR2.2, LVR_DISPENSER.V+, READ_PELLET.2
- net 3.3V: now also R1.2, R2.2, U1.VCC
- net GND: no longer 5-PIN-HEAD.3, D1_OPEN.2, D1_STATE.2, D2_OPEN.2, D2_STATE.2, DISPENSER.GND, DOOR1.GND, DOOR2.GND, IR1.1, IR2.1, LVR_DISPENSER.GND, LVR_FOOD.2, READ_PELLET.1
- net GPIO12: no longer IR1.3
- net GPIO13: no longer IR2.3
- net GPIO16: no longer READ_PELLET.3
- net GPIO17: no longer D2_STATE.1
- net GPIO24: no longer 5-PIN-HEAD.1, D1_OPEN.1
- net GPIO25: no longer 5-PIN-HEAD.2
- net GPIO27: no longer LVR_FOOD.1
- net GPIO4: no longer D1_STATE.1
- net GPIO5: no longer 5-PIN-HEAD.4
- net GPIO6: no longer 5-PIN-HEAD.5, D2_OPEN.1
- net PWM0: no longer DOOR1.SIG
- net PWM1: no longer DISPENSER.SIG
- net PWM13: no longer DOOR2.SIG
- net PWM14: no longer LVR_DISPENSER.SIG
Other:
- note added: "1 + A5 + A4 + A3 + A2 + A1 +A1 + RW"
- note added: "I2C Address ="
- note added: "Open = 0 / Closed = 1"
- note added: "Reverse voltage"
- note added: "protection"
- note removed: "RASPBERRY PI"
- note removed: "SERVO HAT"
