File: Hardware/Electrical/Operant-Front/Operant-Front-Bonsai.brd (EAGLE design)
At the start: 67.9 x 49.2 mm, 14 parts

Commit message: Updated boards
Parts:
- added LED1, LED2, R1, R2, SYNC: (no value), SparkFun-Connectors:1X02
- moved READ_PELLET 10.2 mm to (57.8, 5.08)
Connections:
- new net CONN1: LED1.1, R1.2
- new net CONN2: LED2.1, R2.2
- net GND: now also LED1.2, LED2.2, SYNC.2
- net GPIO19: now also R1.1
- net GPIO20: now also R2.1
- net GPIO23: now also SYNC.1
Routing:
- net GND: track 207.9 -> 231.1 mm
- net GPIO16: track 20.4 -> 38.6 mm
- net GPIO19: track 0.00 -> 16.1 mm
- net GPIO20: track 0.00 -> 15.8 mm
- net GPIO23: track 0.00 -> 7.62 mm
- net CONN2: track 0.00 -> 2.54 mm
- net CONN1: track 0.00 -> 2.54 mm
Other:
- board text added: "10-21-21 Bonsai"
- board text added: "LEDs"
- board text added: "R1"
- board text added: "R2"
- board text removed: "10-14-21 No Bonsai"
