File: Hardware/Electrical/Operant-Front/Operant-Front.brd (EAGLE design)
At the start: 67.9 x 49.2 mm, 34 parts

Commit message: Last commit from PC
Parts:
- removed LVR_1, LVR_10, LVR_11, LVR_12, LVR_13, LVR_14, LVR_15, LVR_16, LVR_2, LVR_3, LVR_4, LVR_5, LVR_6, LVR_7, LVR_8, LVR_9: (no value), SparkFun-Connectors:1X03
Routing:
- net GND: track 202.9 -> 201.3 mm
- net GPIO18: track 30.0 -> 31.3 mm
