File: Hardware/Electrical/Operant-Front/Operant-Front.sch (EAGLE design)
At the start: 53 parts, among them Q1 AOD417, U1 CAT24C32, U2 PCA9685, X1 2.1mm SMT

Commit message: schematics
Parts:
- removed LVR_DOOR1, LVR_DOOR2: SERVO, SparkFun-Electromechanical:SERVO
Connections:
- new net N$1: R1.2, R2.2, U1.VCC
- net +5V: no longer LVR_DOOR1.V+, LVR_DOOR2.V+
- net 3.3V: no longer R1.2, R2.2, U1.VCC
- net GND: no longer LVR_DOOR1.GND, LVR_DOOR2.GND
- net PWM12: no longer LVR_DOOR2.SIG
- net PWM2: no longer LVR_DOOR1.SIG
Other:
- moved on the sheet: DISPENSER, DOOR2, LVR_DISPENSER

Commit message: Schematic
Parts:
- removed 5VIN: 3.5mm term, microbuilder:TERMBLOCK_1X2
- removed C1: 10uF, microbuilder:CAP_CERAMIC0805-NOOUTLINE
- removed C2: (no value), adafruit:CPOL-USE3.5-8
- removed DISPENSER, DOOR1, DOOR2, LVR_DISPENSER: SERVO, SparkFun-Electromechanical:SERVO
- removed JP1, JP2, JP5, JP6: (no value), microbuilder:HEADER-3X04
- removed LED1: GREEN, microbuilder:LED0805_NOOUTLINE
- removed Q1: AOD417, microbuilder:MOSFET-PTO252
- removed R10: 470, microbuilder:RESISTOR_0805MP
- removed R11, R12, R13, R14: 220, microbuilder:RESISTOR_4PACK
- removed R4, R5: 10K, microbuilder:RESISTOR_4PACK
- removed R7: 10K, microbuilder:RESISTOR0805_NOOUTLINE
- removed SJ_A0, SJ_A1, SJ_A2, SJ_A3, SJ_A4, SJ_A5: (no value), microbuilder:SOLDERJUMPERREFLOW_NOPASTE
- removed TP1, TP2, TP3, TP4, TP5, TP6: TPB1,27, testpad:TPB1,27
- removed U2: PCA9685, microbuilder:PCA9685
- removed X1: 2.1mm SMT, microbuilder:DCBARRELSMT_CORRECT
Connections:
- removed net A0: R5G$2.2, SJ_A0.2, TP1.TP, U2.A0
- removed net A1: R5G$1.2, SJ_A1.2, TP2.TP, U2.A1
- removed net A2: R4G$4.2, SJ_A2.2, TP3.TP, U2.A2
- removed net A3: R4G$3.2, SJ_A3.2, TP4.TP, U2.A3
- removed net A4: R4G$2.2, SJ_A4.2, TP5.TP, U2.A4
- removed net A5: R4G$1.2, SJ_A5.2, TP6.TP, U2.A5
- removed net N$24: LED1.C, R10.1
- removed net N$25: JP1.4, R11G$2.2
- removed net N$26: JP1.1, R11G$1.2
- removed net N$27: JP1.7, R11G$3.2
- removed net N$28: JP1.10, R11G$4.2
- removed net N$29: JP2.1, R13G$1.2
- removed net N$30: JP2.4, R13G$2.2
- removed net N$31: JP2.7, R13G$3.2
- removed net N$32: JP2.10, R13G$4.2
- removed net N$33: JP6.10, R14G$4.2
- removed net N$34: JP6.7, R14G$3.2
- removed net N$35: JP6.4, R14G$2.2
- removed net N$36: JP6.1, R14G$1.2
- removed net N$37: JP5.10, R12G$4.2
- removed net N$38: JP5.7, R12G$3.2
- removed net N$40: JP5.4, R12G$2.2
- removed net N$63: JP5.1, R12G$1.2
- removed net OE: R7.1, U2.#OE
- removed net PWM0: DOOR1.SIG, R13G$4.1, U2.PWM0
- removed net PWM1: DISPENSER.SIG, R13G$3.1, U2.PWM1
- removed net PWM10: R14G$2.1, U2.PWM10
- removed net PWM11: R14G$1.1, U2.PWM11
- removed net PWM12: R12G$4.1, U2.PWM12
- removed net PWM13: DOOR2.SIG, R12G$3.1, U2.PWM13
- removed net PWM14: LVR_DISPENSER.SIG, R12G$2.1, U2.PWM14
- removed net PWM15: R12G$1.1, U2.PWM15
- removed net PWM2: R13G$2.1, U2.PWM2
- removed net PWM3: R13G$1.1, U2.PWM3
- removed net PWM4: R11G$4.1, U2.PWM4
- removed net PWM5: R11G$3.1, U2.PWM5
- removed net PWM6: R11G$2.1, U2.PWM6
- removed net PWM7: R11G$1.1, U2.PWM7
- removed net PWM8: R14G$4.1, U2.PWM8
- removed net PWM9: R14G$3.1, U2.PWM9
- removed net PWRIN: 5VIN.1, Q1.D, X1.PWR
- net +5V: no longer C2.+, DISPENSER.V+, DOOR1.V+, DOOR2.V+, JP1.11, JP1.2, JP1.5, JP1.8, JP2.11, JP2.2, JP2.5, JP2.8, JP5.11, JP5.2, JP5.5, JP5.8, JP6.11, JP6.2, JP6.5, JP6.8, LED1.A, LVR_DISPENSER.V+, Q1.S
- net 3.3V: no longer C1.1, SJ_A0.1, SJ_A1.1, SJ_A2.1, SJ_A3.1, SJ_A4.1, SJ_A5.1, U2.VDD
- net GND: no longer 5VIN.2, C1.2, C2.-, DISPENSER.GND, DOOR1.GND, DOOR2.GND, JP1.12, JP1.3, JP1.6, JP1.9, JP2.12, JP2.3, JP2.6, JP2.9, JP5.12, JP5.3, JP5.6, JP5.9, JP6.12, JP6.3, JP6.6, JP6.9, LVR_DISPENSER.GND, Q1.G, R10.2, R4G$1.1, R4G$2.1, R4G$3.1, R4G$4.1, R5G$1.1, R5G$2.1, R7.2, U2.EXTCLK, U2.GND, X1.GND, X1.GNDBREAK
- net SCL: no longer U2.SCL
- net SDA: no longer U2.SDA
Other:
- note removed: "SERVO HAT"
- moved on the sheet: 5-PIN-HEAD, D1_OPEN, D1_STATE, D2_OPEN, D2_STATE, IR1, IR2, LVR_FOOD, READ_PELLET

Commit message: PCB Designs
Parts:
- removed CONN1: HEADER-1X25, microbuilder:HEADER-1X25
- removed R1, R2, R3: 3.9K, microbuilder:RESISTOR0805_NOOUTLINE
- removed RPI1: RASPBERRYPI_BPLUS_HATSLOTS, microbuilder:RASPBERRYPI_BPLUS_HATSLOTS
- removed SJ1: WP, microbuilder:SOLDERJUMPER_CLOSED
- removed U1: CAT24C32, microbuilder:EEPROM_I2C_SOIC8_GENERIC
- added BACK_BOARD_CONN: (no value), SparkFun-Connectors:CONN_04JST-PTH
- added PI_HEADER: (no value), SparkFun-Connectors:CONN_25
- added POWER, SPEAKER: 455-1750-1-ND, SparkFun-Connectors:CONN_03
- D1_OPEN, D1_STATE, D2_OPEN, D2_STATE, LVR_FOOD: device adafruit:JST_2PIN-SMT -> SparkFun-Connectors:CONN_02JST-PTH-2
- IR1, IR2, READ_PELLET: device adafruit:JST_3PIN -> SparkFun-Connectors:CONN_03JST-PTH
Connections:
- removed net 3.3V: R3.2, RPI1.3.3V, RPI1.3.3V@1
- removed net 5.0V: RPI1.5.0V, RPI1.5.0V@1
- removed net EECLK: R2.1, RPI1.EECLK, U1.SCL
- removed net EEDATA: R1.1, RPI1.EEDATA, U1.SDA
- removed net GPIO26: RPI1.GPIO26
- removed net N$1: R1.2, R2.2, U1.VCC
- removed net N$16: R3.1, SJ1.2, U1.WP
- net +5V: now also BACK_BOARD_CONN.1, POWER.3, SPEAKER.2
- net GND: now also BACK_BOARD_CONN.4, D1_OPEN.1, D1_STATE.1, D2_OPEN.1, D2_STATE.1, LVR_FOOD.1, POWER.1, SPEAKER.3; no longer D1_OPEN.2, D1_STATE.2, D2_OPEN.2, D2_STATE.2, LVR_FOOD.2, RPI1.GND, RPI1.GND@1, RPI1.GND@2, RPI1.GND@3, RPI1.GND@4, RPI1.GND@5, RPI1.GND@6, RPI1.GND@7, SJ1.1, U1.A0, U1.A1, U1.A2, U1.GND
- net GPIO12: now also PI_HEADER.20; no longer CONN1.20, RPI1.GPIO12
- net GPIO13: now also PI_HEADER.21; no longer CONN1.21, RPI1.GPIO13
- net GPIO16: now also PI_HEADER.22; no longer CONN1.22, RPI1.GPIO16
- net GPIO17: now also D2_STATE.2, PI_HEADER.6; no longer CONN1.6, D2_STATE.1, RPI1.GPIO17
- net GPIO18: now also BACK_BOARD_CONN.3, PI_HEADER.7; no longer CONN1.7, RPI1.GPIO18
- net GPIO19: now also PI_HEADER.23; no longer CONN1.23, RPI1.GPIO19
- net GPIO20: now also PI_HEADER.24; no longer CONN1.24, RPI1.GPIO20
- net GPIO21: now also PI_HEADER.25, SPEAKER.1; no longer CONN1.25, RPI1.GPIO21
- net GPIO22: now also BACK_BOARD_CONN.2, PI_HEADER.9; no longer CONN1.9, RPI1.GPIO22
- net GPIO23: now also PI_HEADER.10; no longer CONN1.10, RPI1.GPIO23
- net GPIO24: now also D1_OPEN.2, PI_HEADER.11; no longer CONN1.11, D1_OPEN.1, RPI1.GPIO24
- net GPIO25: now also PI_HEADER.12; no longer CONN1.12, RPI1.GPIO25
- net GPIO27: now also LVR_FOOD.2, PI_HEADER.8; no longer CONN1.8, LVR_FOOD.1, RPI1.GPIO27
- net GPIO4: now also D1_STATE.2, PI_HEADER.5; no longer CONN1.5, D1_STATE.1, RPI1.GPIO4
- net GPIO5: now also PI_HEADER.18; no longer CONN1.18, RPI1.GPIO5
- net GPIO6: now also D2_OPEN.2, PI_HEADER.19; no longer CONN1.19, D2_OPEN.1, RPI1.GPIO6
- net RXD: now also PI_HEADER.4; no longer CONN1.4, RPI1.RXD
- net SCL: now also PI_HEADER.2; no longer CONN1.2, RPI1.SCL
- net SDA: now also PI_HEADER.1; no longer CONN1.1, RPI1.SDA
- net SPI_CE0: now also PI_HEADER.16; no longer CONN1.16, RPI1.#SPI_CE0
- net SPI_CE1: now also PI_HEADER.17; no longer CONN1.17, RPI1.#SPI_CE1
- net SPI_MISO: now also PI_HEADER.14; no longer CONN1.14, RPI1.SPI_MISO
- net SPI_MOSI: now also PI_HEADER.13; no longer CONN1.13, RPI1.SPI_MOSI
- net SPI_SCLK: now also PI_HEADER.15; no longer CONN1.15, RPI1.SPI_SCLK
- net TXD: now also PI_HEADER.3; no longer CONN1.3, RPI1.TXD
Other:
- note removed: "RASPBERRY PI"
- moved on the sheet: 5-PIN-HEAD, D1_OPEN, D1_STATE, D2_OPEN, D2_STATE, LVR_FOOD

Commit message: Final version for standard operant board
Parts:
- POWER: value 455-1750-1-ND -> (none)
- SPEAKER: value 455-1750-1-ND -> (none); device SparkFun-Connectors:CONN_03 -> SparkFun-Connectors:CONN_03JST-PTH
Other:
- note added: "Operant Standard"
- moved on the sheet: SPEAKER
Changed lines of the file:
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@@
 </classes>
 <parts>
-<part name="GND6" library="supply1" deviceset="GND" device=""/>
 <part name="GND7" library="supply1" deviceset="GND" device=""/>
 <part name="SUPPLY7" library="supply2" deviceset="+5V" device=""/>
 <part name="5-PIN-HEAD" library="pinhead" library_urn="urn:adsk.eagle:library:325" deviceset="PINHD-1X5" device="" package3d_urn="urn:adsk.eagle:package:22469/2"/>
 <part name="PI_HEADER" library="SparkFun-Connectors" deviceset="CONN_25" device=""/>
-<part name="POWER" library="SparkFun-Connectors" deviceset="CONN_03" device="" value="455-1750-1-ND"/>
-<part name="SPEAKER" library="SparkFun-Connectors" deviceset="CONN_03" device="" value="455-1750-1-ND"/>
+<part name="POWER" library="SparkFun-Connectors" deviceset="CONN_03" device=""/>
 <part name="BACK_BOARD_CONN" library="SparkFun-Connectors" deviceset="CONN_04" device="JST-PTH"/>
 <part name="D1_STATE" library="SparkFun-Connectors" deviceset="CONN_02" device="JST-PTH-2"/>
@@
 <part name="IR2" library="SparkFun-Connectors" deviceset="CONN_03" device="JST-PTH"/>
 <part name="READ_PELLET" library="SparkFun-Connectors" deviceset="CONN_03" device="JST-PTH"/>
+<part name="SPEAKER" library="SparkFun-Connectors" deviceset="CONN_03" device="JST-PTH"/>
 </parts>
 <sheets>
 <sheet>
 <plain>
-<frame x1="170.18" y1="20.32" x2="411.48" y2="200.66" columns="8" rows="5" layer="91"/>
+<frame x1="175.26" y1="22.86" x2="307.34" y2="200.66" columns="8" rows="5" layer="91"/>
+<text x="228.6" y="180.34" size="5.08" layer="91">Operant
+Standard</text>
 </plain>
 <instances>
-<instance part="GND6" gate="1" x="114.3" y="261.62" smashed="yes">
-<attribute name="VALUE" x="111.76" y="259.08" size="1.778" layer="96"/>
-</instance>
 <instance part="GND7" gate="1" x="187.96" y="30.48" smashed="yes">
 <attribute name="VALUE" x="185.42" y="27.94" size="1.778" layer="96"/>
@@
 <attribute name="NAME" x="266.7" y="114.808" size="1.778" layer="95" font="vector"/>
 </instance>
-<instance part="SPEAKER" gate="J$1" x="269.24" y="86.36" smashed="yes">
-<attribute name="VALUE" x="266.7" y="78.994" size="1.778" layer="96" font="vector"/>
-<attribute name="NAME" x="266.7" y="91.948" size="1.778" layer="95" font="vector"/>
-</instance>
 <instance part="BACK_BOARD_CONN" gate="J1" x="271.78" y="63.5" smashed="yes">
 <attribute name="VALUE" x="266.7" y="56.134" size="1.778" layer="96" font="vector"/>
@@
 <attribute name="VALUE" x="218.44" y="66.294" size="1.778" layer="96" font="vector" rot="MR0"/>
 <attribute name="NAME" x="218.44" y="79.248" size="1.778" layer="95" font="vector" rot="MR0"/>
+</instance>
+<instance part="SPEAKER" gate="J$1" x="269.24" y="88.9" smashed="yes">
+<attribute name="VALUE" x="266.7" y="81.534" size="1.778" layer="96" font="vector"/>
+<attribute name="NAME" x="266.7" y="94.488" size="1.778" layer="95" font="vector"/>
 </instance>
 </instances>
@@
 <segment>
 <pinref part="SPEAKER" gate="J$1" pin="3"/>
-<wire x1="276.86" y1="88.9" x2="289.56" y2="88.9" width="0.1524" layer="91"/>
-<label x="284.48" y="88.9" size="1.778" layer="95"/>
+<wire x1="276.86" y1="91.44" x2="289.56" y2="91.44" width="0.1524" layer="91"/>
+<label x="284.48" y="91.44" size="1.778" layer="95"/>
 </segment>
 </net>
@@
 <segment>
 <pinref part="SPEAKER" gate="J$1" pin="1"/>
-<wire x1="276.86" y1="83.82" x2="289.56" y2="83.82" width="0.1524" layer="91"/>
-<label x="281.94" y="83.82" size="1.778" layer="95"/>
+<wire x1="276.86" y1="86.36" x2="289.56" y2="86.36" width="0.1524" layer="91"/>
+<label x="281.94" y="86.36" size="1.778" layer="95"/>
 </segment>
 </net>
@@
 </segment>
 <segment>
-<pinref part="SPEAKER" gate="J$1" pin="2"/>
-<wire x1="276.86" y1="86.36" x2="289.56" y2="86.36" width="0.1524" layer="91"/>
-<label x="284.48" y="86.36" size="1.778" layer="95"/>
-</segment>
-<segment>
 <pinref part="BACK_BOARD_CONN" gate="J1" pin="1"/>
 <wire x1="276.86" y1="60.96" x2="289.56" y2="60.96" width="0.1524" layer="91"/>
 <label x="284.48" y="60.96" size="1.778" layer="95"/>
+</segment>
+<segment>
+<pinref part="SPEAKER" gate="J$1" pin="2"/>
+<wire x1="276.86" y1="88.9" x2="289.56" y2="88.9" width="0.1524" layer="91"/>
+<label x="284.48" y="88.9" size="1.778" layer="95"/>
 </segment>
 </net>
@@
 </drawing>
 <compatibility>
+<note version="6.3" minversion="6.2.2" severity="warning">
+Since Version 6.2.2 text objects can contain more than one line,
+which will not be processed correctly with this version.
+</note>
 <note version="8.2" severity="warning">
 Since Version 8.2, EAGLE supports online libraries. The ids

Commit message: Updated boards
Parts:
- added LED1, LED2, R1, R2, SYNC: (no value), SparkFun-Connectors:CONN_02
Connections:
- new net CONN1: LED1.1, R1.2
- new net CONN2: LED2.1, R2.2
- net GND: now also LED1.2, LED2.2, SYNC.2
- net GPIO19: now also R1.1
- net GPIO20: now also R2.1
- net GPIO23: now also SYNC.1
Changed lines of the file:
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@@
 <part name="READ_PELLET" library="SparkFun-Connectors" deviceset="CONN_03" device="JST-PTH"/>
 <part name="SPEAKER" library="SparkFun-Connectors" deviceset="CONN_03" device="JST-PTH"/>
+<part name="SYNC" library="SparkFun-Connectors" deviceset="CONN_02" device=""/>
+<part name="LED1" library="SparkFun-Connectors" deviceset="CONN_02" device=""/>
+<part name="LED2" library="SparkFun-Connectors" deviceset="CONN_02" device=""/>
+<part name="R1" library="SparkFun-Connectors" deviceset="CONN_02" device=""/>
+<part name="R2" library="SparkFun-Connectors" deviceset="CONN_02" device=""/>
 </parts>
 <sheets>
 <sheet>
 <plain>
-<frame x1="175.26" y1="22.86" x2="307.34" y2="200.66" columns="8" rows="5" layer="91"/>
 <text x="228.6" y="180.34" size="5.08" layer="91">Operant
 Standard</text>
+<frame x1="180.34" y1="-5.08" x2="304.8" y2="200.66" columns="8" rows="5" layer="91"/>
 </plain>
 <instances>
-<instance part="GND7" gate="1" x="187.96" y="30.48" smashed="yes">
-<attribute name="VALUE" x="185.42" y="27.94" size="1.778" layer="96"/>
+<instance part="GND7" gate="1" x="187.96" y="5.08" smashed="yes">
+<attribute name="VALUE" x="185.42" y="2.54" size="1.778" layer="96"/>
 </instance>
 <instance part="SUPPLY7" gate="+5V" x="238.76" y="116.84" smashed="yes">
@@
 <attribute name="VALUE" x="266.7" y="81.534" size="1.778" layer="96" font="vector"/>
 <attribute name="NAME" x="266.7" y="94.488" size="1.778" layer="95" font="vector"/>
+</instance>
+<instance part="SYNC" gate="G$1" x="269.24" y="48.26" smashed="yes">
+<attribute name="VALUE" x="266.7" y="43.434" size="1.778" layer="96" font="vector"/>
+<attribute name="NAME" x="266.7" y="53.848" size="1.778" layer="95" font="vector"/>
+</instance>
+<instance part="LED1" gate="G$1" x="215.9" y="30.48" smashed="yes" rot="MR0">
+<attribute name="VALUE" x="218.44" y="25.654" size="1.778" layer="96" font="vector" rot="MR0"/>
+<attribute name="NAME" x="218.44" y="36.068" size="1.778" layer="95" font="vector" rot="MR0"/>
+</instance>
+<instance part="LED2" gate="G$1" x="215.9" y="17.78" smashed="yes" rot="MR0">
+<attribute name="VALUE" x="218.44" y="12.954" size="1.778" layer="96" font="vector" rot="MR0"/>
+<attribute name="NAME" x="218.44" y="23.368" size="1.778" layer="95" font="vector" rot="MR0"/>
+</instance>
+<instance part="R1" gate="G$1" x="238.76" y="30.48" smashed="yes" rot="MR0">
+<attribute name="VALUE" x="241.3" y="25.654" size="1.778" layer="96" font="vector" rot="MR0"/>
+<attribute name="NAME" x="241.3" y="36.068" size="1.778" layer="95" font="vector" rot="MR0"/>
+</instance>
+<instance part="R2" gate="G$1" x="238.76" y="17.78" smashed="yes" rot="MR0">
+<attribute name="VALUE" x="241.3" y="12.954" size="1.778" layer="96" font="vector" rot="MR0"/>
+<attribute name="NAME" x="241.3" y="23.368" size="1.778" layer="95" font="vector" rot="MR0"/>
 </instance>
 </instances>
@@
 <label x="281.94" y="182.88" size="1.778" layer="95"/>
 </segment>
+<segment>
+<pinref part="R1" gate="G$1" pin="1"/>
+<wire x1="231.14" y1="30.48" x2="223.52" y2="30.48" width="0.1524" layer="91"/>
+<label x="223.52" y="30.48" size="1.778" layer="95"/>
+</segment>
 </net>
 <net name="GND" class="0">
 <segment>
 <pinref part="GND7" gate="1" pin="GND"/>
+<wire x1="187.96" y1="7.62" x2="187.96" y2="20.32" width="0.1524" layer="91"/>
+<wire x1="187.96" y1="20.32" x2="187.96" y2="33.02" width="0.1524" layer="91"/>
 <wire x1="187.96" y1="33.02" x2="187.96" y2="50.8" width="0.1524" layer="91"/>
 <wire x1="187.96" y1="50.8" x2="187.96" y2="71.12" width="0.1524" layer="91"/>
@@
 <wire x1="208.28" y1="71.12" x2="187.96" y2="71.12" width="0.1524" layer="91"/>
 <junction x="187.96" y="71.12"/>
+<pinref part="LED1" gate="G$1" pin="2"/>
+<wire x1="208.28" y1="33.02" x2="187.96" y2="33.02" width="0.1524" layer="91"/>
+<junction x="187.96" y="33.02"/>
+<pinref part="LED2" gate="G$1" pin="2"/>
+<wire x1="208.28" y1="20.32" x2="187.96" y2="20.32" width="0.1524" layer="91"/>
+<junction x="187.96" y="20.32"/>
 </segment>
 <segment>
@@
 <label x="284.48" y="91.44" size="1.778" layer="95"/>
 </segment>
+<segment>
+<pinref part="SYNC" gate="G$1" pin="2"/>
+<wire x1="276.86" y1="50.8" x2="289.56" y2="50.8" width="0.1524" layer="91"/>
+<label x="284.48" y="50.8" size="1.778" layer="95"/>
+</segment>
 </net>
 <net name="TXD" class="0">
@@
 <label x="281.94" y="185.42" size="1.778" layer="95"/>
 </segment>
+<segment>
+<pinref part="R2" gate="G$1" pin="1"/>
+<wire x1="231.14" y1="17.78" x2="223.52" y2="17.78" width="0.1524" layer="91"/>
+<label x="223.52" y="17.78" size="1.778" layer="95"/>
+</segment>
 </net>
 <net name="GPIO21" class="0">
@@
 <wire x1="276.86" y1="149.86" x2="289.56" y2="149.86" width="0.1524" layer="91"/>
 <label x="281.94" y="149.86" size="1.778" layer="95"/>
+</segment>
+<segment>
+<pinref part="SYNC" gate="G$1" pin="1"/>
+<wire x1="276.86" y1="48.26" x2="289.56" y2="48.26" width="0.1524" layer="91"/>
+<label x="281.94" y="48.26" size="1.778" layer="95"/>
 </segment>
 </net>
@@
 </segment>
 </net>
+<net name="CONN1" class="0">
+<segment>
+<pinref part="R1" gate="G$1" pin="2"/>
+<wire x1="231.14" y1="33.02" x2="223.52" y2="33.02" width="0.1524" layer="91"/>
+<label x="223.52" y="33.02" size="1.778" layer="95"/>
+</segment>
+<segment>
+<pinref part="LED1" gate="G$1" pin="1"/>
+<wire x1="208.28" y1="30.48" x2="200.66" y2="30.48" width="0.1524" layer="91"/>
+<label x="200.66" y="30.48" size="1.778" layer="95"/>
+</segment>
+</net>
+<net name="CONN2" class="0">
+<segment>
+<pinref part="R2" gate="G$1" pin="2"/>
+<wire x1="231.14" y1="20.32" x2="223.52" y2="20.32" width="0.1524" layer="91"/>
+<label x="223.52" y="20.32" size="1.778" layer="95"/>
+</segment>
+<segment>
+<pinref part="LED2" gate="G$1" pin="1"/>
+<wire x1="208.28" y1="17.78" x2="200.66" y2="17.78" width="0.1524" layer="91"/>
+<label x="200.66" y="17.78" size="1.778" layer="95"/>
+</segment>
+</net>
