File: Hardware/Electrical/Operant-Front/Operant-Front-Extended.brd (EAGLE design)
At the start: 67.9 x 49.2 mm, 34 parts

Commit message: Extended Board
Parts:
- removed LVR_10, LVR_11, LVR_12, LVR_14, LVR_4, LVR_5, LVR_6, LVR_7, LVR_8, LVR_9: (no value), SparkFun-Connectors:1X03
- added SERVO1, SERVO2: (no value), SparkFun-Connectors:1X03
- moved LVR_16 72.9 mm to (9.53, 8.26), turned to 270 degrees
- moved LVR_15 69.8 mm to (12.1, 8.26), turned to 270 degrees
- moved LVR_13 64.1 mm to (17.1, 8.26), turned to 270 degrees
- moved LVR_3 60.5 mm to (50.2, 8.26), turned to 270 degrees
- moved 5-PIN-HEAD 12.7 mm to (36.8, 38.1)
- moved POWER 12.7 mm to (63.5, 38.1)
- moved R1 12.7 mm to (54.6, 35.6)
- moved R2 12.7 mm to (57.8, 35.6)
- moved D1_OPEN 12.7 mm to (19.1, 27.9)
- moved D1_STATE 12.7 mm to (8.26, 27.9)
- moved IR1 12.7 mm to (46.4, 27.9)
- moved IR2 12.7 mm to (46.4, 17.8)
- moved LVR_1 12.7 mm to (55.2, 8.26)
- moved LVR_2 12.7 mm to (52.7, 8.26)
- moved LVR_FOOD 12.7 mm to (29.8, 27.9)
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Other:
- board size 67.9 x 49.2 mm -> 67.9 x 61.9 mm
- board text added: "10-21-21 Extended"
- board text removed: "10-21-21 No Bonsai"
