File: Hardware/Electrical/Operant-Front/Operant-Front-Extended.sch (EAGLE design)
At the start: 34 parts

Commit message: Extended Board
Parts:
- removed LVR_10, LVR_11, LVR_12, LVR_5, LVR_6, LVR_7, LVR_8, LVR_9: (no value), SparkFun-Connectors:CONN_03
- renumbered LVR_14 to SERVO1, LVR_4 to SERVO2
Changed lines of the file:
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@@
 <part name="LVR_2" library="SparkFun-Connectors" deviceset="CONN_03" device=""/>
 <part name="LVR_3" library="SparkFun-Connectors" deviceset="CONN_03" device=""/>
-<part name="LVR_4" library="SparkFun-Connectors" deviceset="CONN_03" device=""/>
-<part name="LVR_5" library="SparkFun-Connectors" deviceset="CONN_03" device=""/>
-<part name="LVR_6" library="SparkFun-Connectors" deviceset="CONN_03" device=""/>
-<part name="LVR_7" library="SparkFun-Connectors" deviceset="CONN_03" device=""/>
-<part name="LVR_8" library="SparkFun-Connectors" deviceset="CONN_03" device=""/>
-<part name="LVR_9" library="SparkFun-Connectors" deviceset="CONN_03" device=""/>
-<part name="LVR_10" library="SparkFun-Connectors" deviceset="CONN_03" device=""/>
-<part name="LVR_11" library="SparkFun-Connectors" deviceset="CONN_03" device=""/>
-<part name="LVR_12" library="SparkFun-Connectors" deviceset="CONN_03" device=""/>
+<part name="SERVO2" library="SparkFun-Connectors" deviceset="CONN_03" device=""/>
 <part name="LVR_13" library="SparkFun-Connectors" deviceset="CONN_03" device=""/>
-<part name="LVR_14" library="SparkFun-Connectors" deviceset="CONN_03" device=""/>
+<part name="SERVO1" library="SparkFun-Connectors" deviceset="CONN_03" device=""/>
 <part name="LVR_15" library="SparkFun-Connectors" deviceset="CONN_03" device=""/>
 <part name="LVR_16" library="SparkFun-Connectors" deviceset="CONN_03" device=""/>
@@
 <attribute name="NAME" x="284.48" y="38.608" size="1.778" layer="95" font="vector"/>
 </instance>
-<instance part="LVR_4" gate="J$1" x="287.02" y="17.78" smashed="yes">
+<instance part="SERVO2" gate="J$1" x="287.02" y="17.78" smashed="yes">
 <attribute name="VALUE" x="284.48" y="10.414" size="1.778" layer="96" font="vector"/>
 <attribute name="NAME" x="284.48" y="23.368" size="1.778" layer="95" font="vector"/>
-</instance>
-<instance part="LVR_5" gate="J$1" x="322.58" y="33.02" smashed="yes">
-<attribute name="VALUE" x="320.04" y="25.654" size="1.778" layer="96" font="vector"/>
-<attribute name="NAME" x="320.04" y="38.608" size="1.778" layer="95" font="vector"/>
-</instance>
-<instance part="LVR_6" gate="J$1" x="322.58" y="17.78" smashed="yes">
-<attribute name="VALUE" x="320.04" y="10.414" size="1.778" layer="96" font="vector"/>
-<attribute name="NAME" x="320.04" y="23.368" size="1.778" layer="95" font="vector"/>
-</instance>
-<instance part="LVR_7" gate="J$1" x="340.36" y="33.02" smashed="yes">
-<attribute name="VALUE" x="337.82" y="25.654" size="1.778" layer="96" font="vector"/>
-<attribute name="NAME" x="337.82" y="38.608" size="1.778" layer="95" font="vector"/>
-</instance>
-<instance part="LVR_8" gate="J$1" x="340.36" y="17.78" smashed="yes">
-<attribute name="VALUE" x="337.82" y="10.414" size="1.778" layer="96" font="vector"/>
-<attribute name="NAME" x="337.82" y="23.368" size="1.778" layer="95" font="vector"/>
-</instance>
-<instance part="LVR_9" gate="J$1" x="375.92" y="33.02" smashed="yes">
-<attribute name="VALUE" x="373.38" y="25.654" size="1.778" layer="96" font="vector"/>
-<attribute name="NAME" x="373.38" y="38.608" size="1.778" layer="95" font="vector"/>
-</instance>
-<instance part="LVR_10" gate="J$1" x="375.92" y="17.78" smashed="yes">
-<attribute name="VALUE" x="373.38" y="10.414" size="1.778" layer="96" font="vector"/>
-<attribute name="NAME" x="373.38" y="23.368" size="1.778" layer="95" font="vector"/>
-</instance>
-<instance part="LVR_11" gate="J$1" x="393.7" y="33.02" smashed="yes">
-<attribute name="VALUE" x="391.16" y="25.654" size="1.778" layer="96" font="vector"/>
-<attribute name="NAME" x="391.16" y="38.608" size="1.778" layer="95" font="vector"/>
-</instance>
-<instance part="LVR_12" gate="J$1" x="393.7" y="17.78" smashed="yes">
-<attribute name="VALUE" x="391.16" y="10.414" size="1.778" layer="96" font="vector"/>
-<attribute name="NAME" x="391.16" y="23.368" size="1.778" layer="95" font="vector"/>
 </instance>
 <instance part="LVR_13" gate="J$1" x="325.12" y="71.12" smashed="yes">
@@
 <attribute name="NAME" x="322.58" y="76.708" size="1.778" layer="95" font="vector"/>
 </instance>
-<instance part="LVR_14" gate="J$1" x="325.12" y="55.88" smashed="yes">
+<instance part="SERVO1" gate="J$1" x="325.12" y="55.88" smashed="yes">
 <attribute name="VALUE" x="322.58" y="48.514" size="1.778" layer="96" font="vector"/>
 <attribute name="NAME" x="322.58" y="61.468" size="1.778" layer="95" font="vector"/>
